Commit message: Add gripper

File: dobot_rviz/urdf/cr5_robot.urdf (robot description, URDF)
Before this commit: robot cr5_robot, 9 links, 8 joints
Links:
- added link gripper; collision mesh filename=package://dobot_rviz/meshes/cr5/PEGA-100-40.STL scale=0.001 0.001 0.001; visual mesh filename=package://dobot_rviz/meshes/cr5/PEGA-100-40.STL scale=0.001 0.001 0.001
Joints:
- added joint gripper_joint: type fixed, parent Link6, child gripper, origin xyz=0 0 0 rpy=0 0 0
